File: Arduino/PI_DMX_PCB/schaltplan 1.0.brd (EAGLE design)
At the start: 160 x 100 mm, 5 parts, among them IC1 MAX3468EPA, IC2 MAX3468EPA

Commit message: leiterplatte
oszie und max und mega
und iwie anderer kram
Parts:
- removed R2: 1,6k, eagle-ltspice:0204/7
- added C1, C2, C3: (no value), capacitor-wima:C2.5-5
- added IC3: AT90S8515P, atmel:DIL40
- added Q1: (no value), crystal:HC49U-V
- added S1: (no value), switch-dil:DS-01
Connections:
- removed net GND: IC1.5, IC2.5
- removed net VCC: IC1.8, IC2.8
- new net N$10: IC3.9, S1.1
- new net N$11: S1.2, U$1.20
- new net N$2: C3.1, IC1.2, IC1.3, IC1.8, IC2.8, IC3.40, R1.1, U$1.1
- new net N$3: C3.2, R1.2, U$1.9
- new net N$4: C1.2, IC3.19, Q1.1
- new net N$5: C2.2, IC3.18, Q1.2
- new net N$6: C1.1, C2.1, IC3.20
- new net N$9: IC1.5, IC2.2, IC2.3, IC2.5, IC3.4, U$1.6
Changed lines of the file:
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@@
 <attribute name="SPICEPREFIX" value="R" x="57.17" y="79.87" size="1.778" layer="27" rot="R90" display="off"/>
-</element>
-<element name="R2" library="eagle-ltspice" package="0204/7" value="1,6k" x="53.36" y="79.87" rot="R270">
-<attribute name="SPICEMODEL" value="1,6k" x="53.36" y="79.87" size="1.778" layer="27" rot="R270" display="off"/>
-<attribute name="SPICEPREFIX" value="R" x="53.36" y="79.87" size="1.778" layer="27" rot="R270" display="off"/>
 </element>
 <element name="U$1" library="RaspberryPi" package="RASPBERRY-PI_REV1" value="RASPBERRY-PI_REV1" x="52.07" y="69.85"/>
@@
 <attribute name="OC_FARNELL" value="unknown" x="0" y="-6.25" size="1.778" layer="27" display="off"/>
 </element>
+<element name="IC3" library="atmel" package="DIL40" value="AT90S8515P" x="22.5" y="-22.5">
+<attribute name="OC_NEWARK" value="unknown" x="22.5" y="-22.5" size="1.778" layer="27" display="off"/>
+<attribute name="MPN" value="" x="22.5" y="-22.5" size="1.778" layer="27" display="off"/>
+<attribute name="MF" value="" x="22.5" y="-22.5" size="1.778" layer="27" display="off"/>
+<attribute name="OC_FARNELL" value="unknown" x="22.5" y="-22.5" size="1.778" layer="27" display="off"/>
+</element>
+<element name="Q1" library="crystal" package="HC49U-V" value="" x="-1.25" y="-37.5">
+<attribute name="OC_NEWARK" value="unknown" x="-1.25" y="-37.5" size="1.778" layer="27" display="off"/>
+<attribute name="MPN" value="" x="-1.25" y="-37.5" size="1.778" layer="27" display="off"/>
+<attribute name="MF" value="" x="-1.25" y="-37.5" size="1.778" layer="27" display="off"/>
+<attribute name="OC_FARNELL" value="1666969" x="-1.25" y="-37.5" size="1.778" layer="27" display="off"/>
+</element>
+<element name="C1" library="capacitor-wima" package="C2.5-5" value="" x="-13.75" y="-40"/>
+<element name="C2" library="capacitor-wima" package="C2.5-5" value="" x="-22.5" y="-40"/>
+<element name="C3" library="capacitor-wima" package="C2.5-5" value="" x="-31.25" y="-40"/>
+<element name="S1" library="switch-dil" package="DS-01" value="" x="-40" y="-37.5">
+<attribute name="OC_NEWARK" value="unknown" x="-40" y="-37.5" size="1.778" layer="27" display="off"/>
+<attribute name="MPN" value="" x="-40" y="-37.5" size="1.778" layer="27" display="off"/>
+<attribute name="MF" value="" x="-40" y="-37.5" size="1.778" layer="27" display="off"/>
+<attribute name="OC_FARNELL" value="unknown" x="-40" y="-37.5" size="1.778" layer="27" display="off"/>
+</element>
 </elements>
 <signals>
-<signal name="GND">
+<signal name="N$2">
+<contactref element="IC3" pad="40"/>
+<contactref element="U$1" pad="1"/>
+<contactref element="R1" pad="1"/>
+<contactref element="C3" pad="1"/>
+<contactref element="IC2" pad="8"/>
+<contactref element="IC1" pad="2"/>
+<contactref element="IC1" pad="3"/>
+<contactref element="IC1" pad="8"/>
+<wire x1="57.17" y1="76.06" x2="82.13" y2="62.81" width="0" layer="19" extent="1-1"/>
+<wire x1="10.16" y1="91.44" x2="57.17" y2="76.06" width="0" layer="19" extent="1-1"/>
+<wire x1="-3.81" y1="-2.44" x2="10.16" y2="91.44" width="0" layer="19" extent="1-1"/>
+<wire x1="-1.27" y1="-10.06" x2="-3.81" y2="-2.44" width="0" layer="19" extent="1-1"/>
+<wire x1="1.27" y1="-10.06" x2="-1.27" y2="-10.06" width="0" layer="19" extent="1-1"/>
+<wire x1="-1.63" y1="-14.88" x2="-1.27" y2="-10.06" width="0" layer="19" extent="1-1"/>
+<wire x1="-32.52" y1="-40" x2="-1.63" y2="-14.88" width="0" layer="19" extent="1-1"/>
+</signal>
+<signal name="N$3">
+<contactref element="U$1" pad="9"/>
+<contactref element="R1" pad="2"/>
+<contactref element="C3" pad="2"/>
+<wire x1="20.32" y1="91.44" x2="57.17" y2="83.68" width="0" layer="19" extent="1-1"/>
+<wire x1="-29.98" y1="-40" x2="20.32" y2="91.44" width="0" layer="19" extent="1-1"/>
+</signal>
+<signal name="N$4">
+<contactref element="IC3" pad="19"/>
+<contactref element="Q1" pad="1"/>
+<contactref element="C1" pad="2"/>
+<wire x1="-3.663" y1="-37.5" x2="-12.48" y2="-40" width="0" layer="19" extent="1-1"/>
+<wire x1="44.09" y1="-30.12" x2="-3.663" y2="-37.5" width="0" layer="19" extent="1-1"/>
+</signal>
+<signal name="N$5">
+<contactref element="IC3" pad="18"/>
+<contactref element="Q1" pad="2"/>
+<contactref element="C2" pad="2"/>
+<wire x1="1.163" y1="-37.5" x2="-21.23" y2="-40" width="0" layer="19" extent="1-1"/>
+<wire x1="41.55" y1="-30.12" x2="1.163" y2="-37.5" width="0" layer="19" extent="1-1"/>
+</signal>
+<signal name="N$6">
+<contactref element="C2" pad="1"/>
+<contactref element="C1" pad="1"/>
+<contactref element="IC3" pad="20"/>
+<wire x1="-15.02" y1="-40" x2="-23.77" y2="-40" width="0" layer="19" extent="1-1"/>
+<wire x1="46.63" y1="-30.12" x2="-15.02" y2="-40" width="0" layer="19" extent="1-1"/>
+</signal>
+<signal name="N$9">
+<contactref element="IC3" pad="4"/>
+<contactref element="U$1" pad="6"/>
+<contactref element="IC1" pad="5"/>
 <contactref element="IC2" pad="5"/>
-<contactref element="IC1" pad="5"/>
+<contactref element="IC2" pad="3"/>
+<contactref element="IC2" pad="2"/>
+<wire x1="77.05" y1="70.43" x2="79.59" y2="70.43" width="0" layer="19" extent="1-1"/>
+<wire x1="74.51" y1="62.81" x2="77.05" y2="70.43" width="0" layer="19" extent="1-1"/>
+<wire x1="15.24" y1="93.98" x2="77.05" y2="70.43" width="0" layer="19" extent="1-1"/>
 <wire x1="3.81" y1="-2.44" x2="74.51" y2="62.81" width="0" layer="19" extent="1-1"/>
+<wire x1="5.99" y1="-30.12" x2="3.81" y2="-2.44" width="0" layer="19" extent="1-1"/>
 </signal>
-<signal name="VCC">
-<contactref element="IC2" pad="8"/>
-<contactref element="IC1" pad="8"/>
-<wire x1="-3.81" y1="-2.44" x2="82.13" y2="62.81" width="0" layer="19" extent="1-1"/>
+<signal name="N$10">
+<contactref element="IC3" pad="9"/>
+<contactref element="S1" pad="1"/>
+<wire x1="18.69" y1="-30.12" x2="-40" y2="-41.31" width="0" layer="19" extent="1-1"/>
+</signal>
+<signal name="N$11">
+<contactref element="S1" pad="2"/>
+<contactref element="U$1" pad="20"/>
+<wire x1="-40" y1="-33.69" x2="33.02" y2="93.98" width="0" layer="19" extent="1-1"/>
 </signal>
 </signals>
