File: Arduino/PI_DMX_PCB/test1.sch (EAGLE design)
At the start: 7 parts, among them IC2 MAX3468EPA, X1 NC3FD-V-B, X2 NC3MD-V-BAG

Commit message: leiterplatte
oszie und max und mega
und iwie anderer kram
Parts:
- removed PCB1: ARDUINO_NANO, E14_Arduino_revB:ARDUINO_NANO
- removed X1: NC3FD-V-B, con-neutrik_ag:NC3FD-V-B
- removed X2: NC3MD-V-BAG, con-neutrik_ag:NC3MD-V-BAG
- added IC1: MAX3468EPA, maxim:MAX3468EPA
Connections:
- removed net N$1: IC2.DI, PCB1.TX1
- removed net N$10: PCB1.D11, R2.2
- removed net N$11: IC2.VCC, PCB1.5V
- removed net N$12: R1.2, R2.1, U$1.GPIO15,UART0_RXD
- removed net N$13: IC2.GND, PCB1.GND., R1.1, U$1.GND@6, X1.2, X1.G, X2.2, X2.G
- removed net N$14: PCB1.D10, U$1.GPIO14,UART0_TXD
- removed net N$2: IC2.DE, IC2.RE/, PCB1.D2
- removed net N$3: PCB1.VIN, U$1.5V@4
- removed net N$4: IC2.RO, PCB1.RX0
- removed net N$5: IC2.B, X1.1, X2.1
- removed net N$9: IC2.A, X1.3, X2.3
Other:
- moved on the sheet: IC2
Changed lines of the file:
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@@
 </classes>
 <parts>
-<part name="PCB1" library="E14_Arduino_revB" deviceset="ARDUINO_NANO" device=""/>
 <part name="IC2" library="maxim" deviceset="MAX34*" device="PA" technology="68E"/>
 <part name="U$1" library="RaspberryPi" deviceset="RASPBERRY-PI_REV1" device=""/>
-<part name="X1" library="con-neutrik_ag" deviceset="NC3" device="FD-V-B"/>
-<part name="X2" library="con-neutrik_ag" deviceset="NC3" device="MD-V-BAG"/>
 <part name="R1" library="eagle-ltspice" deviceset="R" device="0204/7" value="3,3k">
 <attribute name="SPICEMODEL" value="3,3k"/>
@@
 <attribute name="SPICEMODEL" value="1,6k"/>
 </part>
+<part name="IC1" library="maxim" deviceset="MAX34*" device="PA" technology="68E"/>
 </parts>
 <sheets>
@@
 </plain>
 <instances>
-<instance part="PCB1" gate="G$1" x="-30.48" y="35.56" rot="R270"/>
-<instance part="IC2" gate="G$1" x="15.24" y="25.4"/>
+<instance part="IC2" gate="G$1" x="35.56" y="22.86"/>
 <instance part="U$1" gate="G$1" x="-86.36" y="68.58"/>
-<instance part="X1" gate="G$1" x="134.62" y="25.4"/>
-<instance part="X2" gate="G$1" x="132.08" y="78.74"/>
 <instance part="R1" gate="G$1" x="-40.64" y="86.36">
 <attribute name="SPICEMODEL" x="-50.8" y="86.36" size="1.778" layer="96"/>
@@
 <attribute name="SPICEMODEL" x="-22.86" y="86.36" size="1.778" layer="96"/>
 </instance>
+<instance part="IC1" gate="G$1" x="35.56" y="63.5"/>
 </instances>
 <busses>
 </busses>
 <nets>
-<net name="N$9" class="0">
-<segment>
-<pinref part="X1" gate="G$1" pin="3"/>
-<wire x1="127" y1="25.4" x2="119.38" y2="25.4" width="0.1524" layer="91"/>
-<pinref part="X2" gate="G$1" pin="3"/>
-<wire x1="124.46" y1="78.74" x2="119.38" y2="78.74" width="0.1524" layer="91"/>
-<wire x1="119.38" y1="78.74" x2="119.38" y2="25.4" width="0.1524" layer="91"/>
-<pinref part="IC2" gate="G$1" pin="A"/>
-<junction x="119.38" y="25.4"/>
-<wire x1="35.56" y1="25.4" x2="119.38" y2="25.4" width="0.1524" layer="91"/>
-</segment>
-</net>
-<net name="N$11" class="0">
-<segment>
-<pinref part="IC2" gate="G$1" pin="VCC"/>
-<wire x1="-53.34" y1="25.4" x2="-53.34" y2="0" width="0.1524" layer="91"/>
-<wire x1="-53.34" y1="0" x2="40.64" y2="0" width="0.1524" layer="91"/>
-<wire x1="40.64" y1="0" x2="40.64" y2="38.1" width="0.1524" layer="91"/>
-<wire x1="40.64" y1="38.1" x2="35.56" y2="38.1" width="0.1524" layer="91"/>
-<pinref part="PCB1" gate="G$1" pin="5V"/>
-<wire x1="-48.26" y1="25.4" x2="-53.34" y2="25.4" width="0.1524" layer="91"/>
-</segment>
-</net>
-<net name="N$1" class="0">
-<segment>
-<wire x1="0" y1="17.78" x2="0" y2="20.32" width="0.1524" layer="91"/>
-<pinref part="PCB1" gate="G$1" pin="TX1"/>
-<wire x1="-15.24" y1="17.78" x2="0" y2="17.78" width="0.1524" layer="91"/>
-<pinref part="IC2" gate="G$1" pin="DI"/>
-<wire x1="2.54" y1="20.32" x2="0" y2="20.32" width="0.1524" layer="91"/>
-</segment>
-</net>
-<net name="N$2" class="0">
-<segment>
-<pinref part="IC2" gate="G$1" pin="DE"/>
-<wire x1="-2.54" y1="30.48" x2="-2.54" y2="25.4" width="0.1524" layer="91"/>
-<wire x1="-2.54" y1="25.4" x2="2.54" y2="25.4" width="0.1524" layer="91"/>
-<pinref part="IC2" gate="G$1" pin="RE/"/>
-<wire x1="2.54" y1="30.48" x2="-2.54" y2="30.48" width="0.1524" layer="91"/>
-<junction x="-2.54" y="30.48"/>
-<pinref part="PCB1" gate="G$1" pin="D2"/>
-<wire x1="-2.54" y1="30.48" x2="-2.54" y2="27.94" width="0.1524" layer="91"/>
-<wire x1="-2.54" y1="27.94" x2="-15.24" y2="27.94" width="0.1524" layer="91"/>
-</segment>
-</net>
-<net name="N$4" class="0">
-<segment>
-<pinref part="IC2" gate="G$1" pin="RO"/>
-<wire x1="-5.08" y1="35.56" x2="2.54" y2="35.56" width="0.1524" layer="91"/>
-<pinref part="PCB1" gate="G$1" pin="RX0"/>
-<wire x1="-15.24" y1="20.32" x2="-5.08" y2="20.32" width="0.1524" layer="91"/>
-<wire x1="-5.08" y1="20.32" x2="-5.08" y2="35.56" width="0.1524" layer="91"/>
-</segment>
-</net>
-<net name="N$5" class="0">
-<segment>
-<pinref part="X2" gate="G$1" pin="1"/>
-<wire x1="121.92" y1="81.28" x2="124.46" y2="81.28" width="0.1524" layer="91"/>
-<wire x1="121.92" y1="27.94" x2="121.92" y2="81.28" width="0.1524" layer="91"/>
-<pinref part="X1" gate="G$1" pin="1"/>
-<wire x1="127" y1="27.94" x2="121.92" y2="27.94" width="0.1524" layer="91"/>
-<pinref part="IC2" gate="G$1" pin="B"/>
-<wire x1="121.92" y1="27.94" x2="35.56" y2="27.94" width="0.1524" layer="91"/>
-<wire x1="35.56" y1="27.94" x2="35.56" y2="30.48" width="0.1524" layer="91"/>
-<junction x="121.92" y="27.94"/>
-</segment>
-</net>
-<net name="N$3" class="0">
-<segment>
-<pinref part="U$1" gate="G$1" pin="5V@4"/>
-<wire x1="-58.42" y1="81.28" x2="-53.34" y2="81.28" width="0.1524" layer="91"/>
-<pinref part="PCB1" gate="G$1" pin="VIN"/>
-<wire x1="-48.26" y1="17.78" x2="-50.8" y2="17.78" width="0.1524" layer="91"/>
-<wire x1="-50.8" y1="17.78" x2="-50.8" y2="81.28" width="0.1524" layer="91"/>
-<wire x1="-50.8" y1="81.28" x2="-58.42" y2="81.28" width="0.1524" layer="91"/>
-<junction x="-58.42" y="81.28"/>
-</segment>
-</net>
-<net name="N$10" class="0">
-<segment>
-<wire x1="-17.78" y1="86.36" x2="-10.16" y2="86.36" width="0.1524" layer="91"/>
-<pinref part="PCB1" gate="G$1" pin="D11"/>
-<wire x1="-10.16" y1="86.36" x2="-10.16" y2="50.8" width="0.1524" layer="91"/>
-<wire x1="-10.16" y1="50.8" x2="-15.24" y2="50.8" width="0.1524" layer="91"/>
-<pinref part="R2" gate="G$1" pin="2"/>
-</segment>
-</net>
-<net name="N$12" class="0">
-<segment>
-<pinref part="U$1" gate="G$1" pin="GPIO15,UART0_RXD"/>
-<wire x1="-58.42" y1="73.66" x2="-27.94" y2="73.66" width="0.1524" layer="91"/>
-<pinref part="R2" gate="G$1" pin="1"/>
-<wire x1="-27.94" y1="73.66" x2="-27.94" y2="86.36" width="0.1524" layer="91"/>
-<pinref part="R1" gate="G$1" pin="2"/>
-<wire x1="-27.94" y1="86.36" x2="-35.56" y2="86.36" width="0.1524" layer="91"/>
-<junction x="-27.94" y="86.36"/>
-</segment>
-</net>
-<net name="N$13" class="0">
-<segment>
-<pinref part="R1" gate="G$1" pin="1"/>
-<pinref part="U$1" gate="G$1" pin="GND@6"/>
-<wire x1="-45.72" y1="86.36" x2="-45.72" y2="78.74" width="0.1524" layer="91"/>
-<wire x1="-45.72" y1="78.74" x2="-55.88" y2="78.74" width="0.1524" layer="91"/>
-<pinref part="IC2" gate="G$1" pin="GND"/>
-<pinref part="X1" gate="G$1" pin="G"/>
-<wire x1="-55.88" y1="78.74" x2="-58.42" y2="78.74" width="0.1524" layer="91"/>
-<wire x1="35.56" y1="17.78" x2="45.72" y2="17.78" width="0.1524" layer="91"/>
-<wire x1="45.72" y1="17.78" x2="114.3" y2="17.78" width="0.1524" layer="91"/>
-<wire x1="114.3" y1="17.78" x2="127" y2="17.78" width="0.1524" layer="91"/>
-<wire x1="127" y1="17.78" x2="127" y2="20.32" width="0.1524" layer="91"/>
-<pinref part="X2" gate="G$1" pin="G"/>
-<wire x1="124.46" y1="73.66" x2="114.3" y2="73.66" width="0.1524" layer="91"/>
-<wire x1="114.3" y1="73.66" x2="114.3" y2="17.78" width="0.1524" layer="91"/>
-<junction x="114.3" y="17.78"/>
-<pinref part="PCB1" gate="G$1" pin="GND."/>
-<wire x1="-48.26" y1="20.32" x2="-55.88" y2="20.32" width="0.1524" layer="91"/>
-<wire x1="-55.88" y1="20.32" x2="-58.42" y2="20.32" width="0.1524" layer="91"/>
-<wire x1="-58.42" y1="20.32" x2="-58.42" y2="-5.08" width="0.1524" layer="91"/>
-<wire x1="-58.42" y1="-5.08" x2="45.72" y2="-5.08" width="0.1524" layer="91"/>
-<wire x1="45.72" y1="-5.08" x2="45.72" y2="17.78" width="0.1524" layer="91"/>
-<junction x="45.72" y="17.78"/>
-<wire x1="-55.88" y1="78.74" x2="-55.88" y2="20.32" width="0.1524" layer="91"/>
-<junction x="-55.88" y="78.74"/>
-<junction x="-55.88" y="20.32"/>
-<pinref part="X2" gate="G$1" pin="2"/>
-<wire x1="124.46" y1="76.2" x2="124.46" y2="73.66" width="0.1524" layer="91"/>
-<junction x="124.46" y="73.66"/>
-<pinref part="X1" gate="G$1" pin="2"/>
-<wire x1="127" y1="22.86" x2="127" y2="20.32" width="0.1524" layer="91"/>
-<junction x="127" y="20.32"/>
-</segment>
-</net>
-<net name="N$14" class="0">
-<segment>
-<pinref part="PCB1" gate="G$1" pin="D10"/>
-<wire x1="-7.62" y1="76.2" x2="-7.62" y2="48.26" width="0.1524" layer="91"/>
-<wire x1="-7.62" y1="48.26" x2="-15.24" y2="48.26" width="0.1524" layer="91"/>
-<pinref part="U$1" gate="G$1" pin="GPIO14,UART0_TXD"/>
-<wire x1="-58.42" y1="76.2" x2="-7.62" y2="76.2" width="0.1524" layer="91"/>
-</segment>
-</net>
 </nets>
 </sheet>
